File: IMACS_Keyboard/IMACS_Keyboard.kicad_pcb (KiCad board)
At the start: 2 copper layers, 321.5 x 116.7 mm, 123 parts, among them J1 Keyswitch, K1 Keyswitch, M1 Keyswitch, P1 Keyswitch, Q1 Keyswitch, T1 Keyswitch, U1 SC0915, U2 Keyswitch, X1 Keyswitch, Y1 Keyswitch

Commit message: changed hole position
Routing:
- net COL6: track 285.8 -> 286.9 mm
- net COL5: track 268.4 -> 269.5 mm
Other:
- outline, holes or cut-outs redrawn
Changed lines of the file:
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@@
 	)
 	(gr_circle
-		(center 350 140)
-		(end 351.6 140)
+		(center 350 145)
+		(end 351.6 145)
 		(stroke
 			(width 0.05)
@@
 	)
 	(segment
+		(start 210.5025 98.90125)
+		(end 220.0275 108.42625)
+		(width 0.2)
+		(layer "F.Cu")
+		(net 96)
+	)
+	(segment
+		(start 220.0275 144.40875)
+		(end 220.0275 108.42625)
+		(width 0.2)
+		(layer "F.Cu")
+		(net 96)
+	)
+	(segment
 		(start 359.75 103.34625)
 		(end 357 106.09625)
@@
 	)
 	(segment
-		(start 210.5025 98.90125)
-		(end 220.0275 108.42625)
-		(width 0.2)
-		(layer "F.Cu")
-		(net 96)
-	)
-	(segment
-		(start 357 106.09625)
-		(end 357 141.2625)
-		(width 0.2)
-		(layer "F.Cu")
-		(net 96)
-	)
-	(segment
-		(start 220.0275 144.40875)
-		(end 220.0275 108.42625)
-		(width 0.2)
-		(layer "F.Cu")
-		(net 96)
-	)
-	(segment
 		(start 205.74 70.32625)
 		(end 205.74 84.61375)
@@
 	)
 	(segment
+		(start 357 143)
+		(end 351.78125 148.21875)
+		(width 0.2)
+		(layer "F.Cu")
+		(net 96)
+	)
+	(segment
 		(start 196.215 51.27625)
 		(end 196.215 60.80125)
@@
 	)
 	(segment
-		(start 357 141.2625)
-		(end 350.04375 148.21875)
-		(width 0.2)
-		(layer "F.Cu")
-		(net 96)
-	)
-	(segment
-		(start 350.04375 148.21875)
-		(end 223.8375 148.21875)
-		(width 0.2)
-		(layer "F.Cu")
-		(net 96)
-	)
-	(segment
 		(start 196.215 60.80125)
 		(end 205.74 70.32625)
@@
 		(start 223.8375 148.21875)
 		(end 220.0275 144.40875)
+		(width 0.2)
+		(layer "F.Cu")
+		(net 96)
+	)
+	(segment
+		(start 357 106.09625)
+		(end 357 143)
+		(width 0.2)
+		(layer "F.Cu")
+		(net 96)
+	)
+	(segment
+		(start 351.78125 148.21875)
+		(end 223.8375 148.21875)
 		(width 0.2)
 		(layer "F.Cu")
@@
 	)
 	(segment
-		(start 356.25 104.30625)
-		(end 356.25 141.446814)
+		(start 354.424203 145)
+		(end 351.605453 147.81875)
+		(width 0.2)
+		(layer "F.Cu")
+		(net 97)
+	)
+	(segment
+		(start 239.0775 144.00875)
+		(end 239.0775 108.42625)
 		(width 0.2)
 		(layer "F.Cu")
@@
 	)
 	(segment
-		(start 239.0775 144.00875)
-		(end 239.0775 108.42625)
+		(start 356.25 143.184314)
+		(end 354.434314 145)
+		(width 0.2)
+		(layer "F.Cu")
+		(net 97)
+	)
+	(segment
+		(start 351.605453 147.81875)
+		(end 242.8875 147.81875)
+		(width 0.2)
+		(layer "F.Cu")
+		(net 97)
+	)
+	(segment
+		(start 354.434314 145)
+		(end 354.424203 145)
 		(width 0.2)
 		(layer "F.Cu")
@@
 	)
 	(segment
-		(start 349.878064 147.81875)
-		(end 242.8875 147.81875)
+		(start 242.8875 147.81875)
+		(end 239.0775 144.00875)
 		(width 0.2)
 		(layer "F.Cu")
@@
 	)
 	(segment
-		(start 242.8875 147.81875)
-		(end 239.0775 144.00875)
-		(width 0.2)
-		(layer "F.Cu")
-		(net 97)
-	)
-	(segment
-		(start 356.25 141.446814)
-		(end 349.878064 147.81875)
-		(width 0.2)
-		(layer "F.Cu")
+		(start 356.25 104.30625)
+		(end 356.25 143.184314)
+		(width 0.2)
+		(layer "F.Cu")
